Commit message: Refactor URDF file for my_robot structure

File: src/my_robot_description/urdf/my_robot.urdf.xacro (robot description, xacro)
@@ -22,5 +22,5 @@
         <visual>
             <geometry>
-                <mesh filename="package://my_robot_description/meshes/base_link.stl" scale="0.001 0.001 0.001"/>
+                <mesh filename="package://my_robot_description/meshes/base_link.stl"/>
             </geometry>
             <material name="grey"/>
@@ -28,12 +28,12 @@
         <collision>
             <geometry>
-                <mesh filename="package://my_robot_description/meshes/base_link.stl" scale="0.001 0.001 0.001"/>
+                <mesh filename="package://my_robot_description/meshes/base_link.stl"/>
             </geometry>
         </collision>
     </link>
-    <link name="Link_1">
+    <link name="link_1">
         <visual>
             <geometry>
-                <mesh filename="package://my_robot_description/meshes/link_1.stl" scale="0.001 0.001 0.001"/>
+                <mesh filename="package://my_robot_description/meshes/link_1.stl"/>
             </geometry>
             <material name="blue"/>
@@ -41,12 +41,12 @@
         <collision>
             <geometry>
-                <mesh filename="package://my_robot_description/meshes/link_1.stl" scale="0.001 0.001 0.001"/>
+                <mesh filename="package://my_robot_description/meshes/link_1.stl"/>
             </geometry>
         </collision>
     </link>
-    <link name="Link_2">
+    <link name="link_2">
         <visual>
             <geometry>
-                <mesh filename="package://my_robot_description/meshes/link_2.stl" scale="0.001 0.001 0.001"/>
+                <mesh filename="package://my_robot_description/meshes/link_2.stl"/>
             </geometry>
             <material name="grey"/>
@@ -54,12 +54,25 @@
         <collision>
             <geometry>
-                <mesh filename="package://my_robot_description/meshes/link_2.stl" scale="0.001 0.001 0.001"/>
+                <mesh filename="package://my_robot_description/meshes/link_2.stl"/>
             </geometry>
         </collision>
     </link>
-    <link name="Link_3">
+    <link name="link_3">
         <visual>
             <geometry>
-                <mesh filename="package://my_robot_description/meshes/link_2.stl" scale="0.001 0.001 0.001"/>
+                <mesh filename="package://my_robot_description/meshes/link_3.stl"/>
+            </geometry>
+            <material name="blue"/>
+        </visual>
+        <collision>
+            <geometry>
+                <mesh filename="package://my_robot_description/meshes/link_3.stl"/>
+            </geometry>
+        </collision>
+    </link>
+    <link name="link_4">
+        <visual>
+            <geometry>
+                <mesh filename="package://my_robot_description/meshes/link_4.stl"/>
             </geometry>
             <material name="grey"/>
@@ -67,12 +80,25 @@
         <collision>
             <geometry>
-                <mesh filename="package://my_robot_description/meshes/link_2.stl" scale="0.001 0.001 0.001"/>
+                <mesh filename="package://my_robot_description/meshes/link_4.stl"/>
             </geometry>
         </collision>
     </link>
-    <link name="Link_4">
+    <link name="link_5">
         <visual>
             <geometry>
-                <mesh filename="package://my_robot_description/meshes/link_2.stl" scale="0.001 0.001 0.001"/>
+                <mesh filename="package://my_robot_description/meshes/link_5.stl"/>
+            </geometry>
+            <material name="blue"/>
+        </visual>
+        <collision>
+            <geometry>
+                <mesh filename="package://my_robot_description/meshes/link_5.stl"/>
+            </geometry>
+        </collision>
+    </link>
+    <link name="link_6">
+        <visual>
+            <geometry>
+                <mesh filename="package://my_robot_description/meshes/link_6.stl"/>
             </geometry>
             <material name="grey"/>
@@ -80,37 +106,10 @@
         <collision>
             <geometry>
-                <mesh filename="package://my_robot_description/meshes/link_2.stl" scale="0.001 0.001 0.001"/>
-            </geometry>
-        </collision>
-    </link>
-    <link name="Link_5">
-        <visual>
-            <geometry>
-                <mesh filename="package://my_robot_description/meshes/link_2.stl" scale="0.001 0.001 0.001"/>
-            </geometry>
-            <material name="grey"/>
-        </visual>
-        <collision>
-            <geometry>
-                <mesh filename="package://my_robot_description/meshes/link_2.stl" scale="0.001 0.001 0.001"/>
-            </geometry>
-        </collision>
-    </link>
-    <link name="Link_6">
-        <visual>
-            <geometry>
-                <mesh filename="package://my_robot_description/meshes/link_2.stl" scale="0.001 0.001 0.001"/>
-            </geometry>
-            <material name="grey"/>
-        </visual>
-        <collision>
-            <geometry>
-                <mesh filename="package://my_robot_description/meshes/link_2.stl" scale="0.001 0.001 0.001"/>
+                <mesh filename="package://my_robot_description/meshes/link_6.stl"/>
             </geometry>
         </collision>
     </link>
     <joint name="joint_1" type="revolute">
-        <parent link="Base_link"/>
-        <child link="Link_1"/>
+        <parent link="base_link"/> <child link="link_1"/>
         <origin xyz="0 0 ${d1}" rpy="0 0 0"/>
         <axis xyz="0 0 1"/>
@@ -118,6 +117,6 @@
     </joint>
     <joint name="joint_2" type="revolute">
-        <parent link="Link_1"/>
-        <child link="Link_2"/>
+        <parent link="link_1"/>
+        <child link="link_2"/>
         <origin xyz="${a1} 0 0" rpy="${alpha1} 0 0"/>
         <axis xyz="0 0 1"/>
@@ -125,6 +124,6 @@
     </joint>
     <joint name="joint_3" type="revolute">
-        <parent link="Link_2"/>
-        <child link="Link_3"/>
+        <parent link="link_2"/>
+        <child link="link_3"/>
         <origin xyz="${a2} 0 ${d3}" rpy="${alpha2} 0 0"/>
         <axis xyz="0 0 1"/>
@@ -132,6 +131,6 @@
     </joint>
     <joint name="joint_4" type="revolute">
-        <parent link="Link_3"/>
-        <child link="Link_4"/>
+        <parent link="link_3"/>
+        <child link="link_4"/>
         <origin xyz="${a3} 0 ${d4}" rpy="${alpha3} 0 0"/>
         <axis xyz="0 0 1"/>
@@ -139,8 +138,13 @@
     </joint>
     <joint name="joint_5" type="revolute">
-        <parent link="Link_4"/>
-        <child link="Link_5"/>
-        <origin xyz="${a3} 0 ${d4}" rpy="${alpha3} 0 0"/>
-        <axis xyz="0 0 1"/>
+        <parent link="link_4"/>
+        <child link="link_5"/>
+        <origin xyz="${a4} 0 ${d5}" rpy="${alpha4} 0 0"/> <axis xyz="0 0 1"/>
+        <limit lower="${-pi}" upper="${pi}" effort="100" velocity="1.0"/>
+    </joint>
+    <joint name="joint_6" type="revolute">
+        <parent link="link_5"/>
+        <child link="link_6"/>
+        <origin xyz="${a5} 0 ${d6}" rpy="${alpha5} 0 0"/> <axis xyz="0 0 1"/>
         <limit lower="${-pi}" upper="${pi}" effort="100" velocity="1.0"/>
     </joint>

Commit message: Modify robot URDF properties and link definitions
Updated robot URDF properties, links, and joints with new dimensions and colors.

File: src/my_robot_description/urdf/my_robot.urdf.xacro (robot description, xacro)
@@ -1,150 +1,209 @@
 <?xml version="1.0"?>
 <robot xmlns:xacro="http://www.ros.org/wiki/xacro" name="my_robot">
-    <xacro:property name="d1" value="0.1602" />
-    <xacro:property name="a1" value="0.0812" />
-    <xacro:property name="alpha1" value="${-pi/2}" />
-    <xacro:property name="d2" value="0.0" />
-    <xacro:property name="a2" value="0.2941" />
-    <xacro:property name="alpha2" value="0.0" />
-    <xacro:property name="d3" value="0.0" />
-    <xacro:property name="a3" value="0.0" />
-    <xacro:property name="alpha3" value="${pi/2}" />
-    <xacro:property name="d4" value="0.217" />
+    <xacro:property name="d1" value="0" />
+    <xacro:property name="a1" value="0" />
+    <xacro:property name="alpha1" value="0" />
+    <xacro:property name="d2" value="0.1512" />
+    <xacro:property name="a2" value="0.0641" />
+    <xacro:property name="alpha2" value="${-pi/2}" />
+    <xacro:property name="d3" value="0" />
+    <xacro:property name="a3" value="0.305" />
+    <xacro:property name="alpha3" value="${-pi/2}" />
+    <xacro:property name="d4" value="0.0" />
     <xacro:property name="a4" value="0.0" />
     <xacro:property name="alpha4" value="${-pi/2}" />
-    <xacro:property name="d5" value="0.0" />
+    <xacro:property name="d5" value="0.226" />
     <xacro:property name="a5" value="0.0" />
     <xacro:property name="alpha5" value="${pi/2}" />
-    <xacro:property name="d6" value="0.025" />
+    <xacro:property name="d6" value="0.0" />
     <xacro:property name="a6" value="0.0" />
-    <xacro:property name="alpha6" value="0.0" />
-    <link name="base_link">
-        <visual>
-            <geometry>
-                <mesh filename="package://my_robot_description/meshes/base_link.stl"/>
-            </geometry>
-            <material name="grey"/>
-        </visual>
-        <collision>
-            <geometry>
-                <mesh filename="package://my_robot_description/meshes/base_link.stl"/>
-            </geometry>
-        </collision>
-    </link>
-    <link name="link_1">
-        <visual>
-            <geometry>
-                <mesh filename="package://my_robot_description/meshes/link_1.stl"/>
-            </geometry>
-            <material name="blue"/>
-        </visual>
-        <collision>
-            <geometry>
-                <mesh filename="package://my_robot_description/meshes/link_1.stl"/>
-            </geometry>
-        </collision>
-    </link>
-    <link name="link_2">
-        <visual>
-            <geometry>
-                <mesh filename="package://my_robot_description/meshes/link_2.stl"/>
-            </geometry>
-            <material name="grey"/>
-        </visual>
-        <collision>
-            <geometry>
-                <mesh filename="package://my_robot_description/meshes/link_2.stl"/>
-            </geometry>
-        </collision>
-    </link>
-    <link name="link_3">
-        <visual>
-            <geometry>
-                <mesh filename="package://my_robot_description/meshes/link_3.stl"/>
-            </geometry>
-            <material name="blue"/>
-        </visual>
-        <collision>
-            <geometry>
-                <mesh filename="package://my_robot_description/meshes/link_3.stl"/>
-            </geometry>
-        </collision>
-    </link>
-    <link name="link_4">
-        <visual>
-            <geometry>
-                <mesh filename="package://my_robot_description/meshes/link_4.stl"/>
-            </geometry>
-            <material name="grey"/>
-        </visual>
-        <collision>
-            <geometry>
-                <mesh filename="package://my_robot_description/meshes/link_4.stl"/>
-            </geometry>
-        </collision>
-    </link>
-    <link name="link_5">
-        <visual>
-            <geometry>
-                <mesh filename="package://my_robot_description/meshes/link_5.stl"/>
-            </geometry>
-            <material name="blue"/>
-        </visual>
-        <collision>
-            <geometry>
-                <mesh filename="package://my_robot_description/meshes/link_5.stl"/>
-            </geometry>
-        </collision>
-    </link>
-    <link name="link_6">
-        <visual>
-            <geometry>
-                <mesh filename="package://my_robot_description/meshes/link_6.stl"/>
-            </geometry>
-            <material name="grey"/>
-        </visual>
-        <collision>
-            <geometry>
-                <mesh filename="package://my_robot_description/meshes/link_6.stl"/>
-            </geometry>
-        </collision>
-    </link>
+    <xacro:property name="alpha6" value="${-pi/2}" />
+    <link name="Base_link">
+    <visual>
+      <geometry>
+        <mesh filename="package://my_robot_description/meshes/Base_link.stl" />
+      </geometry>
+      <material name="blue"/>
+    </visual>
+    <collision>
+      <geometry>
+        <mesh filename="package://my_robot_description/meshes/Base_link.stl"/>
+      </geometry>
+    </collision>
+    <inertial>
+      <mass value="7.459715"/>
+      <origin xyz="-0.169292 -0.070267 -0.01062" rpy="0 0 0"/>
+      <inertia
+          ixx="0.0192"   ixy="7.2931e-07"  ixz="0.002723"
+          iyy="0.06688"  iyz="3.6823e-06"
+          izz="0.0718" />
+    </inertial>
+  </link>
+    <link name="Link_1">
+    <visual>
+      <geometry>
+        <mesh filename="package://my_robot_description/meshes/Link_1.stl" />
+      </geometry>
+      <material name="blue"/>
+    </visual>
+    <collision>
+      <geometry>
+        <mesh filename="package://my_robot_description/meshes/Link_1.stl"/>
+      </geometry>
+    </collision>
+    <inertial>
+      <mass value="7.144819"/>
+      <origin xyz="-0.034714 -0.085659 0.09832" rpy="0 0 0"/>
+      <inertia
+          ixx="0.03258"     ixy="0.002621"    ixz="-0.008713"
+          iyy="0.02746"     iyz="0.005571"
+          izz="2.084e+07" />
+    </inertial>
+  </link>
+    <link name="Link_2">
+    <visual>
+      <geometry>
+        <mesh filename="package://my_robot_description/meshes/Link_2.stl" />
+      </geometry>
+      <material name="red"/>
+    </visual>
+    <collision>
+      <geometry>
+        <mesh filename="package://my_robot_description/meshes/Link_2.stl"  />
+      </geometry>
+    </collision>
+    <inertial>
+      <mass value="2.275306"/>
+      <origin xyz="-0.013716 -0.016519 0.02379" rpy="0 0 0"/>
+      <inertia
+          ixx="0.02892"     ixy="-1.36994e-07"  ixz="-3.584117e-06"
+          iyy="0.02943"     iyz="-6.8824154e-05"
+          izz="9.466e+05" />
+    </inertial>
+  </link>
+    <link name="Link_3">
+    <visual>
+      <geometry>
+        <mesh filename="package://my_robot_description/meshes/Link_3.stl"  />
+      </geometry>
+      <material name="green"/>
+    </visual>
+    <collision>
+      <geometry>
+        <mesh filename="package://my_robot_description/meshes/Link_3.stl"/>
+      </geometry>
+    </collision>
+    <inertial>
+      <mass value="1.721937"/>
+      <origin xyz="-0.018038 -0.063262 0.423" rpy="0 0 0"/>
+      <inertia
+          ixx="0.00187"     ixy="-0.0001058"    ixz="-7.1784629e-05"
+          iyy="0.002313"    iyz="-0.0002432"
+          izz="0.001424" />
+    </inertial>
+  </link>
+  <link name="Link_4">
+    <visual>
+      <geometry>
+        <mesh filename="package://my_robot_description/meshes/Link_4.stl" />
+      </geometry>
+      <material name="yellow"/>
+    </visual>
+    <collision>
+      <geometry>
+        <mesh filename="package://my_robot_description/meshes/Link_4.stl" />
+      </geometry>
+    </collision>
+    <inertial>
+      <mass value="2.516104"/>
+      <origin xyz="0.073436 -0.063409 0.446069" rpy="0 0 0"/>
+      <inertia
+          ixx="0.001275"    ixy="-0.001859"    ixz="1.6048041e-05"
+          iyy="0.02139"     iyz="-7.729732e-06"
+          izz="0.02163" />
+    </inertial>
+  </link>
+    <link name="Link_5">
+    <visual>
+      <geometry>
+        <mesh filename="package://my_robot_description/meshes/Link_5.stl"  />
+      </geometry>
+      <material name="purple"/>
+    </visual>
+    <collision>
+      <geometry>
+        <mesh filename="package://my_robot_description/meshes/Link_5.stl"  />
+      </geometry>
+    </collision>
+    <inertial>
+      <mass value="0.737922"/>
+      <origin xyz="0.197942 -0.072188 0.447687" rpy="0 0 0"/>
+      <inertia
+          ixx="0.0002075"   ixy="-2.393396e-06"  ixz="-1.3462959e-05"
+          iyy="0.0003291"   iyz="4.07477e-06"
+          izz="0.0003319" />
+    </inertial>
+  </link>
+    <link name="Link_6">
+    <visual>
+      <geometry>
+        <mesh filename="package://my_robot_description/meshes/Link_6.stl" />
+      </geometry>
+      <material name="orange"/>
+    </visual>
+    <collision>
+      <geometry>
+        <mesh filename="package://my_robot_description/meshes/Link_6.stl" />
+      </geometry>
+    </collision>
+    <inertial>
+      <mass value="0.325456"/>
+      <origin xyz="0.250969 -0.072331 0.446293" rpy="0 0 0"/>
+      <inertia
+          ixx="8.6930674e-05" ixy="-5.851e-09"    ixz="1.6137e-08"
+          iyy="7.1777476e-05" iyz="2.22753e-07"
+          izz="0.0001153" />
+    </inertial>
+  </link>
     <joint name="joint_1" type="revolute">
-        <parent link="base_link"/> <child link="link_1"/>
-        <origin xyz="0 0 ${d1}" rpy="0 0 0"/>
+        <parent link="Base_link"/>
+        <child link="Link_1"/>
+        <origin xyz="0 0 0" rpy="0 0 0"/>
         <axis xyz="0 0 1"/>
         <limit lower="${-pi}" upper="${pi}" effort="100" velocity="1.0"/>
     </joint>
     <joint name="joint_2" type="revolute">
-        <parent link="link_1"/>
-        <child link="link_2"/>
-        <origin xyz="${a1} 0 0" rpy="${alpha1} 0 0"/>
+        <parent link="Link_1"/>
+        <child link="Link_2"/>
+        <origin xyz="${a2} 0.053 ${d2}" rpy="${alpha2} 0 0"/>
         <axis xyz="0 0 1"/>
         <limit lower="${-pi/2}" upper="${pi/2}" effort="100" velocity="1.0"/>
     </joint>
     <joint name="joint_3" type="revolute">
-        <parent link="link_2"/>
-        <child link="link_3"/>
-        <origin xyz="${a2} 0 ${d3}" rpy="${alpha2} 0 0"/>
+        <parent link="Link_2"/>
+        <child link="Link_3"/>
+        <origin xyz="0 -0.305 0" rpy="0 0 ${alpha3}"/>
         <axis xyz="0 0 1"/>
         <limit lower="${-pi}" upper="${pi}" effort="100" velocity="1.0"/>
     </joint>
     <joint name="joint_4" type="revolute">
-        <parent link="link_3"/>
-        <child link="link_4"/>
-        <origin xyz="${a3} 0 ${d4}" rpy="${alpha3} 0 0"/>
+        <parent link="Link_3"/>
+        <child link="Link_4"/>
+        <origin xyz="${a4} 0 ${d4}" rpy="${alpha4} 0 0"/>
         <axis xyz="0 0 1"/>
         <limit lower="${-pi}" upper="${pi}" effort="100" velocity="1.0"/>
     </joint>
     <joint name="joint_5" type="revolute">
-        <parent link="link_4"/>
-        <child link="link_5"/>
-        <origin xyz="${a4} 0 ${d5}" rpy="${alpha4} 0 0"/> <axis xyz="0 0 1"/>
+        <parent link="Link_4"/>
+        <child link="Link_5"/>
+        <origin xyz="${a5} 0 ${d5}" rpy="${alpha5} 0 0"/>
+        <axis xyz="0 0 1"/>
         <limit lower="${-pi}" upper="${pi}" effort="100" velocity="1.0"/>
     </joint>
     <joint name="joint_6" type="revolute">
-        <parent link="link_5"/>
-        <child link="link_6"/>
-        <origin xyz="${a5} 0 ${d6}" rpy="${alpha5} 0 0"/> <axis xyz="0 0 1"/>
+        <parent link="Link_5"/>
+        <child link="Link_6"/>
+        <origin xyz="${a6} 0 ${d6}" rpy="${alpha6} 0 0"/>
+        <axis xyz="0 0 1"/>
         <limit lower="${-pi}" upper="${pi}" effort="100" velocity="1.0"/>
     </joint>
@@ -155,3 +214,18 @@
         <color rgba="0.5 0.5 0.5 1.0"/>
     </material>
+    <material name="red">
+        <color rgba="0.8 0.0 0.0 1.0"/>
+    </material>
+    <material name="green">
+        <color rgba="0.0 0.8 0.0 1.0"/>
+    </material>
+    <material name="yellow">
+        <color rgba="0.8 0.8 0.0 1.0"/>
+    </material>
+    <material name="purple">
+        <color rgba="0.5 0.0 0.8 1.0"/>
+    </material>
+    <material name="orange">
+        <color rgba="1.0 0.5 0.0 1.0"/>
+    </material>
 </robot>
